File: PDC1920/PDC1920.sch (KiCad schematic (older format))
At the start: 9 parts

Commit message: PDC updates
Parts:
- removed J?: Conn_01x20, symbol Connector_Generic:Conn_01x20
- added C3, C6: 1n, Capacitor_SMD:C_0603_1608Metric_Pad1.05x0.95mm_HandSolder, symbol Device:C
- added C4, C5: NP, Capacitor_SMD:C_0603_1608Metric_Pad1.05x0.95mm_HandSolder, symbol Device:C
- added J3: Conn_01x10_Male, Pressure Sensor PDC:3M_N2510-6V0C-RB-WD, symbol Connector:Conn_01x10_Male
- added L1, L2: 0, Inductor_SMD:L_0603_1608Metric_Pad1.05x0.95mm_HandSolder, symbol Device:L
- added R3, R4: 470, Resistor_SMD:R_0603_1608Metric_Pad1.05x0.95mm_HandSolder, symbol Device:R
- added U1, U2, U3: PressureSensor, Pressure Sensor PDC:PressureSensor, symbol Pressure~Sensor~Schematic:PressureSensor
- C1, C2: renamed from C?; footprint (none) -> Capacitor_SMD:C_0603_1608Metric_Pad1.05x0.95mm_HandSolder
- IC1: renamed from IC?; footprint SOIC127P1030X265-18N -> Pressure Sensor PDC:SOIC127P1030X265-18N
- IC2: renamed from IC?; footprint SOT95P237X112-3N -> Pressure Sensor PDC:SOT95P237X112-3N
- J1: renamed from J?; footprint (none) -> Pressure Sensor PDC:37946364
- J2: renamed from J?; footprint (none) -> Connector_PinHeader_2.54mm:PinHeader_1x06_P2.54mm_Vertical_SMD_Pin1Right
- R1, R2: renamed from R?; footprint (none) -> Resistor_SMD:R_0603_1608Metric_Pad1.05x0.95mm_HandSolder
Connections:
- net labels added: MISO, RX_Pic, SCLK, SS0, SS1, SS2, SS3, SS4, SS5, TX_Pic
- wire segments 17 -> 51
Other:
- moved on the sheet: C1, C2, IC1, IC2, J1, J2, R1, R2

Commit message: Clearance changes
Parts:
- U1, U2, U3: symbol Pressure~Sensor~Schematic:PressureSensor -> PDC1920-rescue:PressureSensor-Pressure~Sensor~Schematic
Changed lines of the file:
@@
 Connection ~ 4400 4550
 $Comp
-L Pressure~Sensor~Schematic:PressureSensor U2
+L PDC1920-rescue:PressureSensor-Pressure~Sensor~Schematic U2
 U 1 1 5E2B9A49
 P 5650 2700
@@
 $EndComp
 $Comp
-L Pressure~Sensor~Schematic:PressureSensor U3
+L PDC1920-rescue:PressureSensor-Pressure~Sensor~Schematic U3
 U 1 1 5E2B9E78
 P 5650 3250
@@
 SS4
 $Comp
-L Pressure~Sensor~Schematic:PressureSensor U1
+L PDC1920-rescue:PressureSensor-Pressure~Sensor~Schematic U1
 U 1 1 5E2B91FC
 P 5650 2100
